Commit message: changed urdfs

File: dinova_description/urdf/dinova.xacro (robot description, xacro)
@@ -4,4 +4,5 @@
     <xacro:arg name="load_gripper" default="true"/>
     <xacro:arg name="dingo_real_urdf" default="true"/>
+    <xacro:arg name="lidar" default="true"/>
     <!-- Add dingo -->
     <xacro:if value="$(arg dingo_real_urdf)">
@@ -32,9 +33,24 @@
         </joint>
     </xacro:if>
-    <!-- Connection between dingo and kinova -->
-    <joint name="$(arg robot_id)arm_mount_joint" type="fixed">
-        <origin rpy="0 0 0" xyz="0 0 0"/>
-        <parent link="$(arg robot_id)front_b_mount"/>
-        <child link="$(arg robot_id)kinova_base_link"/>
-    </joint>
+    <!-- Check lidar option -->
+    <xacro:if value="$(arg lidar)">
+        <!-- Connection between dingo and kinova -->
+        <joint name="$(arg robot_id)arm_mount_joint" type="fixed">
+            <origin rpy="0 0 0" xyz="0 0 0.314"/>
+            <parent link="$(arg robot_id)front_b_mount"/>
+            <child link="$(arg robot_id)kinova_base_link"/>
+        </joint>
+        <xacro:include filename="$(find velodyne_description)/urdf/VLP-16.urdf.xacro"/>
+        <xacro:VLP-16 parent="mid_mount" name="velodyne" topic="/velodyne_points" hz="10" samples="440" gpu="false" min_range="0.4" >
+            <origin xyz="0 0 0" rpy="0 0 0" />
+        </xacro:VLP-16>
+    </xacro:if>
+    <xacro:unless value="$(arg lidar)">
+        <!-- Connection between dingo and kinova -->
+        <joint name="$(arg robot_id)arm_mount_joint" type="fixed">
+            <origin rpy="0 0 0" xyz="0 0 0"/>
+            <parent link="$(arg robot_id)front_b_mount"/>
+            <child link="$(arg robot_id)kinova_base_link"/>
+        </joint>
+    </xacro:unless>
 </robot>

Commit message: update

File: dinova_description/urdf/dinova.xacro (robot description, xacro)
@@ -5,4 +5,5 @@
     <xacro:arg name="dingo_real_urdf" default="true"/>
     <xacro:arg name="lidar" default="true"/>
+    <xacro:property name="platform_height" value="0.34" />
     <!-- Add dingo -->
     <xacro:if value="$(arg dingo_real_urdf)">
@@ -35,14 +36,43 @@
     <!-- Check lidar option -->
     <xacro:if value="$(arg lidar)">
+        <xacro:include filename="$(find velodyne_description)/urdf/VLP-16.urdf.xacro"/>
+        <xacro:VLP-16 parent="$(arg robot_id)front_b_mount" name="$(arg robot_id)velodyne" topic="/velodyne_points" hz="10" samples="440" gpu="false" min_range="0.4" >
+            <origin xyz="0 0 0" rpy="0 0 0" />
+        </xacro:VLP-16>
+        <!-- Metal platform -->
+        <link name="$(arg robot_id)platform_link">
+            <visual>
+            <origin rpy="0 0 0" xyz="0 0 ${platform_height/2.0}"/>
+            <geometry>
+                <cylinder length="${platform_height}" radius="0.08"/>
+            </geometry>
+            <material name="gray">
+                <color rgba="0.1 0.1 0.1 0.8"/>
+            </material>
+            </visual>
+            <collision>
+                <origin rpy="0 0 0" xyz="0 0 ${platform_height/2.0}"/>
+                <geometry>
+                    <cylinder length="${platform_height}" radius="0.08"/>
+                </geometry>
+            </collision>
+            <inertial>
+            <origin rpy="0 0 0" xyz="0 0 0"/>
+            <mass value="0.4"/>
+            <inertia ixx="0.0003234" ixy="0" ixz="0" iyy="0.0003234" iyz="0" izz="0.0004901"/>
+            </inertial>
+         </link>
+        <!-- Connection between dingo and kinova -->
+        <joint name="$(arg robot_id)platform_mount_joint" type="fixed">
+            <origin rpy="0 0 0" xyz="0 0 0"/>
+            <parent link="$(arg robot_id)front_b_mount"/>
+            <child link="$(arg robot_id)platform_link"/>
+        </joint>
         <!-- Connection between dingo and kinova -->
         <joint name="$(arg robot_id)arm_mount_joint" type="fixed">
-            <origin rpy="0 0 0" xyz="0 0 0.314"/>
+            <origin rpy="0 0 0" xyz="0 0 ${platform_height}"/>
             <parent link="$(arg robot_id)front_b_mount"/>
             <child link="$(arg robot_id)kinova_base_link"/>
         </joint>
-        <xacro:include filename="$(find velodyne_description)/urdf/VLP-16.urdf.xacro"/>
-        <xacro:VLP-16 parent="mid_mount" name="velodyne" topic="/velodyne_points" hz="10" samples="440" gpu="false" min_range="0.4" >
-            <origin xyz="0 0 0" rpy="0 0 0" />
-        </xacro:VLP-16>
     </xacro:if>
     <xacro:unless value="$(arg lidar)">

Commit message: add lidar option

File: dinova_description/urdf/dinova.xacro (robot description, xacro)
@@ -5,5 +5,5 @@
     <xacro:arg name="dingo_real_urdf" default="true"/>
     <xacro:arg name="lidar" default="true"/>
-    <xacro:property name="platform_height" value="0.34" />
+    <xacro:property name="platform_height" value="0.314" />
     <!-- Add dingo -->
     <xacro:if value="$(arg dingo_real_urdf)">
@@ -36,8 +36,4 @@
     <!-- Check lidar option -->
     <xacro:if value="$(arg lidar)">
-        <xacro:include filename="$(find velodyne_description)/urdf/VLP-16.urdf.xacro"/>
-        <xacro:VLP-16 parent="$(arg robot_id)front_b_mount" name="$(arg robot_id)velodyne" topic="/velodyne_points" hz="10" samples="440" gpu="false" min_range="0.4" >
-            <origin xyz="0 0 0" rpy="0 0 0" />
-        </xacro:VLP-16>
         <!-- Metal platform -->
         <link name="$(arg robot_id)platform_link">
@@ -63,5 +59,5 @@
             </inertial>
          </link>
-        <!-- Connection between dingo and kinova -->
+        <!-- Connection between dingo and platform -->
         <joint name="$(arg robot_id)platform_mount_joint" type="fixed">
             <origin rpy="0 0 0" xyz="0 0 0"/>
@@ -75,4 +71,8 @@
             <child link="$(arg robot_id)kinova_base_link"/>
         </joint>
+        <!-- <xacro:include filename="$(find velodyne_description)/urdf/VLP-16.urdf.xacro"/>
+        <xacro:VLP-16 parent="$(arg robot_id)front_b_mount" name="$(arg robot_id)velodyne" topic="/$(arg robot_id)/velodyne_points" hz="10" samples="440" gpu="false" min_range="0.4" >
+            <origin xyz="0 0 0" rpy="0 0 0" />
+        </xacro:VLP-16> -->
     </xacro:if>
     <xacro:unless value="$(arg lidar)">

Commit message: Update lidar stack height

File: dinova_description/urdf/dinova.xacro (robot description, xacro)
@@ -5,5 +5,5 @@
     <xacro:arg name="dingo_real_urdf" default="true"/>
     <xacro:arg name="lidar" default="true"/>
-    <xacro:property name="platform_height" value="0.314" />
+    <xacro:property name="platform_height" value="0.279" />
     <!-- Add dingo -->
     <xacro:if value="$(arg dingo_real_urdf)">
@@ -67,5 +67,5 @@
         <!-- Connection between dingo and kinova -->
         <joint name="$(arg robot_id)arm_mount_joint" type="fixed">
-            <origin rpy="0 0 0" xyz="0 0 ${platform_height}"/>
+            <origin rpy="0 0 0" xyz="0.0399 0 ${platform_height}"/>
             <parent link="$(arg robot_id)front_b_mount"/>
             <child link="$(arg robot_id)kinova_base_link"/>

Commit message: fix: calibrated models

File: dinova_description/urdf/dinova.xacro (robot description, xacro)
@@ -5,4 +5,6 @@
     <xacro:arg name="dingo_real_urdf" default="true"/>
     <xacro:arg name="lidar" default="true"/>
+    <xacro:arg name="robot_name" default="dingo1"/>
+    <xacro:property name="robot_name" value="$(arg robot_name)"/>
     <xacro:property name="platform_height" value="0.279" />
     <!-- Add dingo -->
@@ -21,6 +23,12 @@
     </xacro:unless>
     <!-- Add kinova -->
-    <xacro:include filename="$(find dinova_description)/urdf/kinova_macro.xacro"/>
-    <xacro:kinova prefix="$(arg robot_id)"/>
+    <xacro:if value="${robot_name == 'dingo1'}">
+        <xacro:include filename="$(find dinova_description)/urdf/kinova1_macro.xacro"/>
+        <xacro:kinova prefix="${robot_id}"/>
+    </xacro:if>
+    <xacro:if value="${robot_name == 'dingo2'}">
+        <xacro:include filename="$(find dinova_description)/urdf/kinova2_macro.xacro"/>
+        <xacro:kinova prefix="$(arg robot_id)"/>
+    </xacro:if>
     <!-- Add kinova gripper -->
     <xacro:if value="$(arg load_gripper)">

File: dinova_description/urdf/kinova.xacro (robot description, xacro)
@@ -3,7 +3,15 @@
     <xacro:arg name="arm_id" default="" />
     <xacro:arg name="load_gripper" default="true"/>
+    <xacro:arg name="robot_name" default="dingo1"/>
+    <xacro:property name="robot_name" value="$(arg robot_name)"/>
     <!-- Add kinova -->
-    <xacro:include filename="$(find dinova_description)/urdf/kinova_macro.xacro"/>
-    <xacro:kinova prefix="$(arg arm_id)"/>
+    <xacro:if value="${robot_name == 'dingo1'}">
+        <xacro:include filename="$(find dinova_description)/urdf/kinova1_macro.xacro"/>
+        <xacro:kinova prefix="${arm_id}"/>
+    </xacro:if>
+    <xacro:if value="${robot_name == 'dingo2'}">
+        <xacro:include filename="$(find dinova_description)/urdf/kinova2_macro.xacro"/>
+        <xacro:kinova prefix="$(arg arm_id)"/>
+    </xacro:if>
     <!-- Add kinova gripper -->
     <xacro:if value="$(arg load_gripper)">
