Commit message: fixed urdf

File: dinova_description/urdf/dingo_omni_macro.xacro (robot description, xacro)
@@ -83,5 +83,5 @@
             <origin rpy="0 0 0" xyz="0 0 0"/>
             <geometry>
-                <mesh filename="package://dingo_kinova_description/urdf/meshes/base/omni_chassis.dae"/>
+                <mesh filename="package://dinova_description/urdf/meshes/base/omni_chassis.dae"/>
             </geometry>
             <material name="dark_grey"/>
@@ -90,5 +90,5 @@
             <origin xyz="0 0 0"/>
             <geometry>
-                <mesh filename="package://dingo_kinova_description/urdf/meshes/base/omni_chassis_collision.stl"/>
+                <mesh filename="package://dinova_description/urdf/meshes/base/omni_chassis_collision.stl"/>
             </geometry>
         </collision>

File: dinova_description/urdf/dinova.xacro (robot description, xacro)
@@ -8,8 +8,14 @@
         <xacro:include filename="$(find dinova_description)/urdf/real_dingo-o.urdf.xacro" />
     </xacro:if>
-    <xacro:if value="$(not arg dingo_real_urdf)">
-        <param name="robot_description" command="$(find xacro)/xacro '$(find dinova_description)/urdf/dingo_omni.xacro'
-                                                dingo_id:=$(arg robot_id)"/>
-    </xacro:if>
+    <xacro:unless value="$(arg dingo_real_urdf)">
+        <xacro:include filename="$(find dinova_description)/urdf/dingo_omni_macro.xacro"/>
+        <xacro:dingo_omni prefix="$(arg robot_id)"/>
+        <link name="world"/>
+        <joint name="$(arg robot_id)world_link" type="fixed">
+            <origin rpy="0 0 0" xyz="0 0 0"/>
+            <parent link="world"/>
+            <child link="$(arg robot_id)base_link"/>
+        </joint>
+    </xacro:unless>
     <!-- Add kinova -->
     <xacro:include filename="$(find dinova_description)/urdf/kinova_macro.xacro"/>

File: dinova_description/urdf/kinova_gripper_macro.xacro (robot description, xacro)
@@ -130,29 +130,29 @@
     </joint>
     <!-- right_finger_tip_joint -->
-    <joint name="${prefix}right_finger_tip_joint" type="revolute">
+    <joint name="${prefix}right_finger_tip_joint" type="fixed">
         <origin xyz="-0.045636 0.020423 0" rpy="0 0 0" />
         <parent link="${prefix}right_finger_prox_link" />
         <child link="${prefix}right_finger_dist_link" />
         <axis xyz="0 0 1" />
-        <limit lower="-0.50" upper="0.21" effort="1000" velocity="1000" /> <!--limit lower="-1.03" upper="0.21" effort="1000" velocity="1000" /-->
-        <mimic joint="${prefix}right_finger_bottom_joint" multiplier="-0.676" offset="0.149" />
+        <!-- <limit lower="-0.50" upper="0.21" effort="1000" velocity="1000" />  -->
+        <!-- <mimic joint="${prefix}right_finger_bottom_joint" multiplier="-0.676" offset="0.149" /> -->
     </joint>
     <!-- left_finger_bottom_joint  -->
-    <joint name="${prefix}left_finger_bottom_joint" type="revolute">
+    <joint name="${prefix}left_finger_bottom_joint" type="fixed">
         <origin xyz="0 0.0305 0.070003" rpy="0 1.5708 0" />
         <parent link="${prefix}gripper_base_link" />
         <child link="${prefix}left_finger_prox_link" />
         <axis xyz="0 0 1" />
-        <limit lower="-0.96" upper="0.09" effort="1000" velocity="1000" />
-        <mimic joint="${prefix}right_finger_bottom_joint" multiplier="-1.0" offset="0.0" />
+        <!-- <limit lower="-0.96" upper="0.09" effort="1000" velocity="1000" /> -->
+        <!-- <mimic joint="${prefix}right_finger_bottom_joint" multiplier="-1.0" offset="0.0" /> -->
     </joint>
     <!-- left_finger_tip_joint -->
-    <joint name="${prefix}left_finger_tip_joint" type="revolute">
+    <joint name="${prefix}left_finger_tip_joint" type="fixed">
         <origin xyz="-0.045636 -0.020423 6.9901E-05" rpy="0 0 0" />
         <parent link="${prefix}left_finger_prox_link" />
         <child link="${prefix}left_finger_dist_link" />
         <axis xyz="0 0 -1" />
-        <limit lower="-0.50" upper="0.21" effort="1000" velocity="1000" /> <!--limit lower="-1.03" upper="0.21" effort="1000" velocity="1000" /-->
-        <mimic joint="${prefix}right_finger_bottom_joint" multiplier="-0.676" offset="0.149" />
+        <!-- <limit lower="-0.50" upper="0.21" effort="1000" velocity="1000" />  -->
+        <!-- <mimic joint="${prefix}right_finger_bottom_joint" multiplier="-0.676" offset="0.149" /> -->
     </joint>
 </xacro:macro>

Commit message: fix: removing 0.03 from the urdf

File: dinova_description/urdf/dingo_omni_macro.xacro (robot description, xacro)
@@ -52,5 +52,5 @@
         <parent link="${prefix}base_link"/>
         <child link="${prefix}base_link_x"/>
-        <origin rpy="0 0 0" xyz="0 0 0.03"/>
+        <origin rpy="0 0 0" xyz="0 0 0.0"/>
         <axis xyz="1 0 0"/>
         <dynamics damping="100.0"/>

Commit message: Adding z-offset between base_link and first link to avoid a collision, according to solution suggestion to fix #43

File: dinova_description/urdf/dingo_omni_macro.xacro (robot description, xacro)
@@ -52,5 +52,5 @@
         <parent link="${prefix}base_link"/>
         <child link="${prefix}base_link_x"/>
-        <origin rpy="0 0 0" xyz="0 0 0.0"/>
+        <origin rpy="0 0 0" xyz="0 0 0.03"/>
         <axis xyz="1 0 0"/>
         <dynamics damping="100.0"/>
