Commit message: fix: unifying urdfs

File: dinova_control/config/dinova.urdf (robot description, URDF)
Before this commit: robot dingo_kinova, 22 links, 21 joints
Links:
- added link arm_orientation_helper_link
- added link front_left_wheel_link, mass 0.4; collision cylinder length=0.05 radius=0.05; visual cylinder length=0.05 radius=0.05
- added link front_right_wheel_link, mass 0.4; collision cylinder length=0.05 radius=0.05; visual cylinder length=0.05 radius=0.05
- added link rear_left_wheel_link, mass 0.4; collision cylinder length=0.05 radius=0.05; visual cylinder length=0.05 radius=0.05
- added link rear_right_wheel_link, mass 0.4; collision cylinder length=0.05 radius=0.05; visual cylinder length=0.05 radius=0.05
Joints:
- added joint arm_orientation_helper_joint: type fixed, parent arm_dummy_link, child arm_orientation_helper_link, origin xyz=0 0.1 0 rpy=0 0 0, axis 0 0 0
- added joint front_left_wheel: type fixed, parent chassis_link, child front_left_wheel_link, origin xyz=0.285 0.2104 0.035145 rpy=0 0 0, axis 0 1 0
- added joint front_right_wheel: type fixed, parent chassis_link, child front_right_wheel_link, origin xyz=0.285 -0.2104 0.035145 rpy=0 0 0, axis 0 1 0
- added joint rear_left_wheel: type fixed, parent chassis_link, child rear_left_wheel_link, origin xyz=-0.285 0.2104 0.035145 rpy=0 0 0, axis 0 1 0
- added joint rear_right_wheel: type fixed, parent chassis_link, child rear_right_wheel_link, origin xyz=-0.285 -0.2104 0.035145 rpy=0 0 0, axis 0 1 0
- joint omni_joint_x: origin xyz=0 0 0.03 rpy=0 0 0 -> xyz=0 0 0 rpy=0 0 0

File: dinova_control/config/dinova_lidar.urdf (robot description, URDF)
Before this commit: robot dingo_kinova, 22 links, 25 joints
Links:
- added link arm_orientation_helper_link
- added link front_left_wheel_link, mass 0.4; collision cylinder length=0.05 radius=0.05; visual cylinder length=0.05 radius=0.05
- added link front_right_wheel_link, mass 0.4; collision cylinder length=0.05 radius=0.05; visual cylinder length=0.05 radius=0.05
- added link rear_left_wheel_link, mass 0.4; collision cylinder length=0.05 radius=0.05; visual cylinder length=0.05 radius=0.05
- added link rear_right_wheel_link, mass 0.4; collision cylinder length=0.05 radius=0.05; visual cylinder length=0.05 radius=0.05
Joints:
- added joint arm_orientation_helper_joint: type fixed, parent arm_dummy_link, child arm_orientation_helper_link, origin xyz=0 0.1 0 rpy=0 0 0, axis 0 0 0
- joint omni_joint_x: origin xyz=0 0 0.03 rpy=0 0 0 -> xyz=0 0 0 rpy=0 0 0

Commit message: in-process version, fk in urdf calibrated for dingo2

File: dinova_control/config/dinova.urdf (robot description, URDF)
Before this commit: robot dingo_kinova, 27 links, 26 joints
Joints:
- joint arm_joint_1: origin xyz=0 0 0.12825 rpy=0 0 0 -> xyz=-1.8836019394079857e-16 -3.688218839160853e-17 0.12825000000000078 rpy=-2.746893142615157e-05 -0.0012876966269176834 -3.4078623335807743e-16
- joint arm_joint_2: origin xyz=0 -0.03 0.115 rpy=1.5708 0 0 -> xyz=-0.0005014484308504022 -0.029343454485041668 0.11500000000000155 rpy=1.581263130895373 0.015120261949270858 1.5164839538784716e-05
- joint arm_joint_3: origin xyz=0 0.28 0 rpy=-3.1416 0 0 -> xyz=0.004095913096920563 0.28293673179772627 -0.0006561462132585497 rpy=-3.1460688147415032 -0.013928343995075362 -0.01397495853756151
- joint arm_joint_4: origin xyz=0 -0.14 0.02 rpy=1.5708 0 0 -> xyz=0.001465691695560486 -0.1409451077317066 0.020698873181334607 rpy=1.570135251499924 0.00020755089686141798 0.013771183766511014
- joint arm_joint_5: origin xyz=0.0285 0 0.105 rpy=0 1.5708 0 -> xyz=0.028307136985665976 -0.0007740663723995084 0.1059664426831494 rpy=0.00016848106903807688 1.566674528420962 -0.0001763473975477907
- joint arm_joint_6: origin xyz=-0.105 0 0.0285 rpy=0 -1.5708 0 -> xyz=-0.111504270439627 0.002536337273228278 0.02831137395835149 rpy=-0.0016434779097823941 -1.5685481245804054 -0.0016434820817590162

File: dinova_control/config/dinova_lidar.urdf (robot description, URDF)
Before this commit: robot dingo_kinova, 27 links, 26 joints
Joints:
- joint arm_joint_1: origin xyz=0 0 0.12825 rpy=0 0 0 -> xyz=-1.8836019394079857e-16 -3.688218839160853e-17 0.12825000000000078 rpy=-2.746893142615157e-05 -0.0012876966269176834 -3.4078623335807743e-16
- joint arm_joint_2: origin xyz=0 -0.03 0.115 rpy=1.5708 0 0 -> xyz=-0.0005014484308504022 -0.029343454485041668 0.11500000000000155 rpy=1.581263130895373 0.015120261949270858 1.5164839538784716e-05
- joint arm_joint_3: origin xyz=0 0.28 0 rpy=-3.1416 0 0 -> xyz=0.004095913096920563 0.28293673179772627 -0.0006561462132585497 rpy=-3.1460688147415032 -0.013928343995075362 -0.01397495853756151
- joint arm_joint_4: origin xyz=0 -0.14 0.02 rpy=1.5708 0 0 -> xyz=0.001465691695560486 -0.1409451077317066 0.020698873181334607 rpy=1.570135251499924 0.00020755089686141798 0.013771183766511014
- joint arm_joint_5: origin xyz=0.0285 0 0.105 rpy=0 1.5708 0 -> xyz=0.028307136985665976 -0.0007740663723995084 0.1059664426831494 rpy=0.00016848106903807688 1.566674528420962 -0.0001763473975477907
- joint arm_joint_6: origin xyz=-0.105 0 0.0285 rpy=0 -1.5708 0 -> xyz=-0.111504270439627 0.002536337273228278 0.02831137395835149 rpy=-0.0016434779097823941 -1.5685481245804054 -0.0016434820817590162

File: dinova_description/urdf/kinova_macro.xacro (robot description, xacro)
@@ -158,5 +158,5 @@
     <!-- Joint 1 -->
     <joint name="${prefix}joint_1" type="revolute">
-        <origin xyz="0 0 0.12825" rpy="0 0 0" />
+        <origin rpy="-2.746893142615157e-05 -0.0012876966269176834 -3.4078623335807743e-16" xyz="-1.8836019394079857e-16 -3.688218839160853e-17 0.12825000000000078" />
         <parent link="${prefix}kinova_base_link" />
         <child link="${prefix}shoulder_link" />
@@ -166,5 +166,5 @@
     <!-- Joint 2 -->
     <joint name="${prefix}joint_2" type="revolute">
-        <origin xyz="0 -0.03 0.115" rpy="1.5708 0 0" />
+        <origin rpy="1.581263130895373 0.015120261949270858 1.5164839538784716e-05" xyz="-0.0005014484308504022 -0.029343454485041668 0.11500000000000155" />
         <parent link="${prefix}shoulder_link" />
         <child link="${prefix}arm_link" />
@@ -174,5 +174,5 @@
     <!-- Joint 3 -->
     <joint name="${prefix}joint_3" type="revolute">
-        <origin xyz="0 0.28 0" rpy="-3.1416 0 0" />
+        <origin rpy="-3.1460688147415032 -0.013928343995075362 -0.01397495853756151" xyz="0.004095913096920563 0.28293673179772627 -0.0006561462132585497" />
         <parent link="${prefix}arm_link" />
         <child link="${prefix}forearm_link" />
@@ -182,5 +182,5 @@
     <!-- Joint 4 -->
     <joint name="${prefix}joint_4" type="revolute">
-        <origin xyz="0 -0.14 0.02" rpy="1.5708 0 0" />
+        <origin rpy="1.570135251499924 0.00020755089686141798 0.013771183766511014" xyz="0.001465691695560486 -0.1409451077317066 0.020698873181334607" />
         <parent link="${prefix}forearm_link" />
         <child link="${prefix}lower_wrist_link" />
@@ -190,5 +190,5 @@
     <!-- Joint 5 -->
     <joint name="${prefix}joint_5" type="revolute">
-        <origin xyz="0.0285 0 0.105" rpy="0 1.5708 0" />
+        <origin rpy="0.00016848106903807688 1.566674528420962 -0.0001763473975477907" xyz="0.028307136985665976 -0.0007740663723995084 0.1059664426831494" />
         <parent link="${prefix}lower_wrist_link" />
         <child link="${prefix}upper_wrist_link" />
@@ -198,5 +198,5 @@
     <!-- Joint 6 -->
     <joint name="${prefix}joint_6" type="revolute">
-        <origin xyz="-0.105 0 0.0285" rpy="0 -1.5708 0" />
+        <origin rpy="-0.0016434779097823941 -1.5685481245804054 -0.0016434820817590162" xyz="-0.111504270439627 0.002536337273228278 0.02831137395835149" />
         <parent link="${prefix}upper_wrist_link" />
         <child link="${prefix}end_effector_link" />
@@ -216,5 +216,5 @@
     <!-- Tool frame used by the arm -->
    <joint name="${prefix}tool_frame_joint" type="fixed">
-        <origin rpy="0 0 0" xyz="0 0 0.130"/>
+        <origin rpy="0 0 0" xyz="0 0 0.07"/>
         <parent link="${prefix}dummy_link"/>
         <child link="${prefix}tool_frame"/>
