Commit message: fix: using only urdf file from the dingo2

File: dinova_control/config/dingo1_dinova.urdf (robot description, URDF)
Before this commit: robot dingo_kinova, 27 links, 26 joints
Joints:
- joint arm_joint_1: origin xyz=4.988843730662458e-16 -8.173728747909104e-16 0.12824999999999917 rpy=0.0009351385662122073 -1.7366916249849798e-05 -5.512221427531898e-16 -> xyz=-1.8836019394079857e-16 -3.688218839160853e-17 0.12825000000000078 rpy=-2.746893142615157e-05 -0.0012876966269176834 -3.4078623335807743e-16
- joint arm_joint_2: origin xyz=-0.0058803889029462025 -0.029075673583809532 0.11499999999999895 rpy=1.5679382876528443 -0.00436691600857366 0.0001764117326825226 -> xyz=-0.0005014484308504022 -0.029343454485041668 0.11500000000000155 rpy=1.581263130895373 0.015120261949270858 1.5164839538784716e-05
- joint arm_joint_3: origin xyz=-0.00673912346628402 0.2691539807248412 -0.0009252864181610817 rpy=-3.154678419482146 0.012439231759643923 0.002480483516040656 -> xyz=0.004095913096920563 0.28293673179772627 -0.0006561462132585497 rpy=-3.1460688147415032 -0.013928343995075362 -0.01397495853756151
- joint arm_joint_4: origin xyz=-9.697889813732241e-05 -0.13382178071023465 0.021150995396657605 rpy=1.5746001594078056 -0.003718901462378342 -0.002466978281634551 -> xyz=0.001465691695560486 -0.1409451077317066 0.020698873181334607 rpy=1.570135251499924 0.00020755089686141798 0.013771183766511014
- joint arm_joint_5: origin xyz=0.026208819642660044 0.0007609408542277129 0.09881770371083187 rpy=-0.0037007621700123157 1.5733596667368124 0.003706625514882694 -> xyz=0.028307136985665976 -0.0007740663723995084 0.1059664426831494 rpy=0.00016848106903807688 1.566674528420962 -0.0001763473975477907
- joint arm_joint_6: origin xyz=-0.10556672972644801 -0.0012619470520149226 0.02623037375104344 rpy=-0.0024151465343667487 -1.570783400862489 -0.0024151465346838436 -> xyz=-0.111504270439627 0.002536337273228278 0.02831137395835149 rpy=-0.0016434779097823941 -1.5685481245804054 -0.0016434820817590162

File: dinova_control/config/dingo1_dinova_lidar.urdf (robot description, URDF)
Before this commit: robot dingo_kinova, 27 links, 26 joints
Joints:
- joint arm_joint_1: origin xyz=4.988843730662458e-16 -8.173728747909104e-16 0.12824999999999917 rpy=0.0009351385662122073 -1.7366916249849798e-05 -5.512221427531898e-16 -> xyz=-1.8836019394079857e-16 -3.688218839160853e-17 0.12825000000000078 rpy=-2.746893142615157e-05 -0.0012876966269176834 -3.4078623335807743e-16
- joint arm_joint_2: origin xyz=-0.0058803889029462025 -0.029075673583809532 0.11499999999999895 rpy=1.5679382876528443 -0.00436691600857366 0.0001764117326825226 -> xyz=-0.0005014484308504022 -0.029343454485041668 0.11500000000000155 rpy=1.581263130895373 0.015120261949270858 1.5164839538784716e-05
- joint arm_joint_3: origin xyz=-0.00673912346628402 0.2691539807248412 -0.0009252864181610817 rpy=-3.154678419482146 0.012439231759643923 0.002480483516040656 -> xyz=0.004095913096920563 0.28293673179772627 -0.0006561462132585497 rpy=-3.1460688147415032 -0.013928343995075362 -0.01397495853756151
- joint arm_joint_4: origin xyz=-9.697889813732241e-05 -0.13382178071023465 0.021150995396657605 rpy=1.5746001594078056 -0.003718901462378342 -0.002466978281634551 -> xyz=0.001465691695560486 -0.1409451077317066 0.020698873181334607 rpy=1.570135251499924 0.00020755089686141798 0.013771183766511014
- joint arm_joint_5: origin xyz=0.026208819642660044 0.0007609408542277129 0.09881770371083187 rpy=-0.0037007621700123157 1.5733596667368124 0.003706625514882694 -> xyz=0.028307136985665976 -0.0007740663723995084 0.1059664426831494 rpy=0.00016848106903807688 1.566674528420962 -0.0001763473975477907
- joint arm_joint_6: origin xyz=-0.10556672972644801 -0.0012619470520149226 0.02623037375104344 rpy=-0.0024151465343667487 -1.570783400862489 -0.0024151465346838436 -> xyz=-0.111504270439627 0.002536337273228278 0.02831137395835149 rpy=-0.0016434779097823941 -1.5685481245804054 -0.0016434820817590162

File: dinova_description/urdf/kinova1_macro.xacro (robot description, xacro)
@@ -158,5 +158,5 @@
     <!-- Joint 1 -->
     <joint name="${prefix}joint_1" type="revolute">
-        <origin rpy="0.0009351385662122073 -1.7366916249849798e-05 -5.512221427531898e-16" xyz="4.988843730662458e-16 -8.173728747909104e-16 0.12824999999999917" />
+        <origin rpy="-2.746893142615157e-05 -0.0012876966269176834 -3.4078623335807743e-16" xyz="-1.8836019394079857e-16 -3.688218839160853e-17 0.12825000000000078" />
         <parent link="${prefix}kinova_base_link" />
         <child link="${prefix}shoulder_link" />
@@ -166,5 +166,5 @@
     <!-- Joint 2 -->
     <joint name="${prefix}joint_2" type="revolute">
-        <origin rpy="1.5679382876528443 -0.00436691600857366 0.0001764117326825226" xyz="-0.0058803889029462025 -0.029075673583809532 0.11499999999999895" />
+        <origin rpy="1.581263130895373 0.015120261949270858 1.5164839538784716e-05" xyz="-0.0005014484308504022 -0.029343454485041668 0.11500000000000155" />
         <parent link="${prefix}shoulder_link" />
         <child link="${prefix}arm_link" />
@@ -174,5 +174,5 @@
     <!-- Joint 3 -->
     <joint name="${prefix}joint_3" type="revolute">
-        <origin rpy="-3.154678419482146 0.012439231759643923 0.002480483516040656" xyz="-0.00673912346628402 0.2691539807248412 -0.0009252864181610817" />
+        <origin rpy="-3.1460688147415032 -0.013928343995075362 -0.01397495853756151" xyz="0.004095913096920563 0.28293673179772627 -0.0006561462132585497" />
         <parent link="${prefix}arm_link" />
         <child link="${prefix}forearm_link" />
@@ -182,5 +182,5 @@
     <!-- Joint 4 -->
     <joint name="${prefix}joint_4" type="revolute">
-        <origin rpy="1.5746001594078056 -0.003718901462378342 -0.002466978281634551" xyz="-9.697889813732241e-05 -0.13382178071023465 0.021150995396657605" />
+        <origin rpy="1.570135251499924 0.00020755089686141798 0.013771183766511014" xyz="0.001465691695560486 -0.1409451077317066 0.020698873181334607" />
         <parent link="${prefix}forearm_link" />
         <child link="${prefix}lower_wrist_link" />
@@ -190,5 +190,5 @@
     <!-- Joint 5 -->
     <joint name="${prefix}joint_5" type="revolute">
-        <origin rpy="-0.0037007621700123157 1.5733596667368124 0.003706625514882694" xyz="0.026208819642660044 0.0007609408542277129 0.09881770371083187" />
+        <origin rpy="0.00016848106903807688 1.566674528420962 -0.0001763473975477907" xyz="0.028307136985665976 -0.0007740663723995084 0.1059664426831494" />
         <parent link="${prefix}lower_wrist_link" />
         <child link="${prefix}upper_wrist_link" />
@@ -198,5 +198,5 @@
     <!-- Joint 6 -->
     <joint name="${prefix}joint_6" type="revolute">
-        <origin rpy="-0.0024151465343667487 -1.570783400862489 -0.0024151465346838436" xyz="-0.10556672972644801 -0.0012619470520149226 0.02623037375104344" />
+        <origin rpy="-0.0016434779097823941 -1.5685481245804054 -0.0016434820817590162" xyz="-0.111504270439627 0.002536337273228278 0.02831137395835149" />
         <parent link="${prefix}upper_wrist_link" />
         <child link="${prefix}end_effector_link" />
